Commit message: Add arguments to support the new gazebo

File: tiago_pro_description/robots/tiago_pro.urdf.xacro (robot description, xacro)
@@ -12,5 +12,5 @@
   limitations under the License.
 -->
-<robot xmlns:xacro="http://ros.org/wiki/xacro" name="tiago_pro">
+<robot xmlns:xacro="http://ros.org/wiki/xacro" xmlns:gz="http://gazebosim.org/schema" name="tiago_pro">
   <!-- ARGUMENTS -->
   <!-- no-laser, sick-571-->
@@ -323,4 +323,4 @@
   </xacro:if>
   <!-- ROS 2 Control -->
-  <xacro:tiago_pro_ros2_control use_sim_time="$(arg use_sim_time)" has_teleop_arms="${has_teleop_arms}"/>
+  <xacro:tiago_pro_ros2_control use_sim_time="$(arg use_sim_time)" has_teleop_arms="${has_teleop_arms}" gazebo_version="${gazebo_version}"/>
 </robot>

File: tiago_pro_description/ros2_control/ros2_control.urdf.xacro (robot description, xacro)
@@ -105,5 +105,5 @@
     <xacro:ros2_control_head_joint name="head_2" reduction="1.0" offset_value="${head_2_joint_offset}" />
   </xacro:macro>
-  <xacro:macro name="tiago_pro_ros2_control" params="use_sim_time:=^|false has_teleop_arms:=^|false">
+  <xacro:macro name="tiago_pro_ros2_control" params="use_sim_time:=^|false has_teleop_arms:=^|false gazebo_version:=^|classic">
     <xacro:arg name="arm_type_left" default="tiago-pro"/>
     <xacro:arg name="arm_type_right" default="tiago-pro"/>
@@ -149,11 +149,25 @@
       <!-- Init the ROS 2 control gazebo interface -->
       <gazebo>
-        <plugin filename="libgazebo_ros2_control.so" name="gazebo_ros2_control">
-          <parameters>$(find tiago_pro_description)/ros2_control/gazebo_controller_manager_cfg.yaml</parameters>
-        </plugin>
+        <xacro:if value="${gazebo_version == 'classic'}">
+          <plugin filename="libgazebo_ros2_control.so" name="gazebo_ros2_control">
+            <parameters>$(find tiago_pro_description)/ros2_control/gazebo_controller_manager_cfg.yaml</parameters>
+          </plugin>
+        </xacro:if>
+        <xacro:if value="${gazebo_version == 'gazebo'}">
+          <plugin filename="gz_ros2_control-system" name="gz_ros2_control::GazeboSimROS2ControlPlugin">
+            <robot_param>robot_description</robot_param>
+            <robot_param_node>robot_state_publisher</robot_param_node>
+            <parameters>$(find tiago_pro_description)/ros2_control/gazebo_controller_manager_cfg.yaml</parameters>
+          </plugin>
+        </xacro:if>
       </gazebo>
       <ros2_control name="ros2_control_gazebo_system" type="system">
         <hardware>
-          <plugin>gazebo_ros2_control/GazeboSystem</plugin>
+          <xacro:if value="${gazebo_version == 'classic'}">
+            <plugin>gazebo_ros2_control/GazeboSystem</plugin>
+          </xacro:if>
+          <xacro:if value="${gazebo_version == 'gazebo'}">
+            <plugin>gz_ros2_control/GazeboSimSystem</plugin>
+          </xacro:if>
         </hardware>
         <!-- wheels -->
@@ -185,7 +199,18 @@
         <!-- CAN system -->
         <ros2_control name="ros2_control_tiago_pro_system_can" type="system" rw_rate="100">
+          <!-- Execution env config -->
           <hardware>
-            <plugin>robot_control/RobotControl</plugin>
-            <param name="group">can</param>
+            <xacro:if value="${use_sim_time}">
+              <xacro:if value="${gazebo_version == 'classic'}">
+                <plugin>gazebo_ros2_control/GazeboSystem</plugin>
+              </xacro:if>
+              <xacro:if value="${gazebo_version == 'gazebo'}">
+                <plugin>gz_ros2_control/GazeboSimSystem</plugin>
+              </xacro:if>
+            </xacro:if>
+            <xacro:unless value="${use_sim_time}">
+              <plugin>robot_control/RobotControl</plugin>
+              <param name="group">can</param>
+            </xacro:unless>
           </hardware>
           <!-- wheels -->
@@ -196,6 +221,16 @@
       <ros2_control name="ros2_control_tiago_pro_system_dynamixel" type="system" rw_rate="100">
         <hardware>
-          <plugin>robot_control/RobotControl</plugin>
-          <param name="group">dynamixel</param>
+          <xacro:if value="${use_sim_time}">
+            <xacro:if value="${gazebo_version == 'classic'}">
+              <plugin>gazebo_ros2_control/GazeboSystem</plugin>
+            </xacro:if>
+            <xacro:if value="${gazebo_version == 'gazebo'}">
+              <plugin>gz_ros2_control/GazeboSimSystem</plugin>
+            </xacro:if>
+          </xacro:if>
+          <xacro:unless value="${use_sim_time}">
+            <plugin>robot_control/RobotControl</plugin>
+            <param name="group">dynamixel</param>
+          </xacro:unless>
         </hardware>
         <!-- head -->
@@ -205,10 +240,20 @@
       <ros2_control name="ros2_control_tiago_pro_system_ethercat" type="system" rw_rate="1000">
         <hardware>
+          <xacro:if value="${use_sim_time}">
+            <xacro:if value="${gazebo_version == 'classic'}">
+              <plugin>gazebo_ros2_control/GazeboSystem</plugin>
+            </xacro:if>
+            <xacro:if value="${gazebo_version == 'gazebo'}">
+              <plugin>gz_ros2_control/GazeboSimSystem</plugin>
+            </xacro:if>
+          </xacro:if>
+          <xacro:unless value="${use_sim_time}">
           <plugin>robot_control/RobotControl</plugin>
-          <param name="group">ethercat</param>
-          <param name="error_protection">true</param>
-          <param name="idle_mode_on_stop">true</param>
-          <param name="expose_collision_interface">true</param>
-          <param name="expose_safety_interface">true</param>
+            <param name="group">ethercat</param>
+            <param name="error_protection">true</param>
+            <param name="idle_mode_on_stop">true</param>
+            <param name="expose_collision_interface">true</param>
+            <param name="expose_safety_interface">true</param>
+          </xacro:unless>
         </hardware>
         <!-- arms -->

File: tiago_pro_description/urdf/torso/torso.ros2_control.xacro (robot description, xacro)
@@ -16,5 +16,7 @@
     <joint name="${name}_joint">
       <command_interface name="position" />
-      <command_interface name="velocity" />
+      <xacro:if value="${gazebo_version == 'classic'}">
+        <command_interface name="velocity" />
+      </xacro:if>
       <state_interface name="position" />
       <state_interface name="velocity" />
