Commit message: Add safety controller to prevent the torso to get stuck in simulation with a small epsilon

File: tiago_pro_description/urdf/torso/torso.urdf.xacro (robot description, xacro)
@@ -95,4 +95,12 @@
       </collision>
     </link>
+    <!-- TODO: set lower limit back to 0 when moving to Gazebo Harmonic or ROS 2 Jazzy -->
+    <!-- See https://github.com/gazebosim/gz-sim/issues/1684 for more information -->
+    <xacro:if value="${gazebo_version == 'classic'}">
+      <xacro:property name="torso_lower_limit" value="0.0"/>
+    </xacro:if>
+    <xacro:if value="${gazebo_version == 'gazebo'}">
+      <xacro:property name="torso_lower_limit" value="-1e-3"/>
+    </xacro:if>
     <joint name="${name}_lift_joint" type="prismatic">
       <origin xyz="0 0 0.5545" rpy="0 0 0" />
@@ -100,5 +108,5 @@
       <child link="${name}_lift_link" />
       <axis xyz="0 0 1" />
-      <limit effort="2000" lower="0" upper="0.35" velocity="${torso_max_vel}" />
+      <limit effort="2000" lower="${torso_lower_limit}" upper="0.35" velocity="${torso_max_vel}" />
       <calibration rising="0.0" />
       <dynamics damping="1000" />
